File: PCBs/TAStm32.sch (EAGLE design)
At the start: 23 parts, among them J1 ZX62D-B-5PA8, P1 RJHSE-5381, P1_DEBUG 6_PIN_SERIAL_CABLEPTH, P2 RJHSE-5381, P2_DEBUG 6_PIN_SERIAL_CABLEPTH, U1 STM32F446RET6

Commit message: works with new pin assignments
Parts:
- removed C9: 25pF, eagle-ltspice:C
- added C1: 4.7uF, eagle-ltspice:C
- C3: value 4.7uF -> 25pF
- renumbered C10 to C5, C11 to C6, C12 to C7, C8 to C2
Connections:
- net GND: now also C1.2, C3.1; no longer C3.2, C9.1
- net N$6: now also C1.1; no longer C3.1
- net P1_CLOCK: now also U1.PC0/SAI1_MCLK_B/OTG_HS_ULPI_STP/FMC_SDNWE/EVENTOUT; no longer U1.PC2/SPI2_MISO/OTG_HS_ULPI_DIR/FMC_SDNE0/EVENTOUT
- net P1_D0: now also U1.PC3/SPI2_MOSI/I2S2_SD/OTG_HS_ULPI_NXT/FMC_SDCKE0/EVENTOUT; no longer U1.PA8/MCO1/TIM1_CH1/I2C3_SCL/USART1_CK/OTG_FS_SOF/EVENTOUT
- net P1_D1: now also U1.PC2/SPI2_MISO/OTG_HS_ULPI_DIR/FMC_SDNE0/EVENTOUT; no longer U1.PC3/SPI2_MOSI/I2S2_SD/OTG_HS_ULPI_NXT/FMC_SDCKE0/EVENTOUT
- net P2_CLOCK: now also U1.PC5/USART3_RX/SPDIFRX_IN3/FMC_SDCKE0/EVENTOUT; no longer U1.PC0/SAI1_MCLK_B/OTG_HS_ULPI_STP/FMC_SDNWE/EVENTOUT
- net P2_D0: now also U1.PC8/TRACED0/TIM3_CH3/TIM8_CH3/UART5_RTS/USART6_CK/SDIO_D0/DCMI_D2/EVENTOUT; no longer U1.PC7/TIM3_CH2/TIM8_CH2/FMPI2C1_SDA/SPI2_SCK/I2S2_CK/I2S3_MCK/SPDIFRX_IN1/USART6_RX/SDIO_D7/DCMI_D1/EVENTOUT
- net P2_D1: now also U1.PC7/TIM3_CH2/TIM8_CH2/FMPI2C1_SDA/SPI2_SCK/I2S2_CK/I2S3_MCK/SPDIFRX_IN1/USART6_RX/SDIO_D7/DCMI_D1/EVENTOUT; no longer U1.PC8/TRACED0/TIM3_CH3/TIM8_CH3/UART5_RTS/USART6_CK/SDIO_D0/DCMI_D2/EVENTOUT
- net P2_D2: now also U1.PC9/MCO2/TIM3_CH4/TIM8_CH4/I2C3_SDA/I2S_CKIN/UART5_CTS/QUADSPI_BK1_IO0/SDIO_D1/DCMI_D3/EVENTOUT; no longer U1.PC6/TIM3_CH1/TIM8_CH1/FMPI2C1_SCL/I2S2_MCK/USART6_TX/SDIO_D6/DCMI_D0/EVENTOUT
- net P2_LATCH: now also U1.PC6/TIM3_CH1/TIM8_CH1/FMPI2C1_SCL/I2S2_MCK/USART6_TX/SDIO_D6/DCMI_D0/EVENTOUT; no longer U1.PC9/MCO2/TIM3_CH4/TIM8_CH4/I2C3_SDA/I2S_CKIN/UART5_CTS/QUADSPI_BK1_IO0/SDIO_D1/DCMI_D3/EVENTOUT
- net XTAL2: now also C3.2; no longer C9.2
Other:
- moved on the sheet: C3
