File: PCB and Case/TAStm32_v3.brd (EAGLE design)
At the start: 47 x 83.1 mm, 22 parts, among them J1 ZX62D-B-5PA8, P1_DEBUG SAMTEC-TSM-106-01-X-SVJ, P2_DEBUG SAMTEC-TSM-106-01-X-SVJ, U1 STM32F446RET6

Commit message: fixed capacitor C7 value
Parts:
- C7: value 100nF -> 4.7uF
Changed lines of the file:
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@@
 <attribute name="SPICEPREFIX" value="C" x="17.09" y="39.9316" size="1.778" layer="27" rot="R270" display="off"/>
 </element>
-<element name="C7" library="rcl" library_urn="urn:adsk.eagle:library:334" package="C0805K" package3d_urn="urn:adsk.eagle:package:23681/2" value="100nF" x="14.04" y="45.0916" smashed="yes">
+<element name="C7" library="rcl" library_urn="urn:adsk.eagle:library:334" package="C0805K" package3d_urn="urn:adsk.eagle:package:23681/2" value="4.7uF" x="14.04" y="45.0916" smashed="yes">
 <attribute name="NAME" x="10.89" y="45.6016" size="0.6096" layer="25" font="vector" ratio="15" rot="R270"/>
 <attribute name="POPULARITY" value="52" x="14.04" y="45.0916" size="1.778" layer="27" display="off"/>
