File: PCB and Case/TAStm32_v4.brd (EAGLE design)
At the start: 100 x 50 mm, 55 parts, among them CN1 330pF, CN2 330pF, CN3 330pF, CN4 330pF, IC1 74LVC3G17DP, IC2 74LVC3G17DP, IC3 74AXP4T245, IC4 74AXP4T245, J1 ZX62D-B-5PA8, J10 RJSSE538002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

Commit message: Set input filter caps to DNP
Parts:
- CN1, CN2: value 330pF -> DNP
- S1, S2, S3, S4: value 3-1825910-1_SWITCHN -> 3-1825910-1
Changed lines of the file:
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@@
 <attribute name="VALUE" x="57.456" y="14.028" size="1.27" layer="27" rot="R270"/>
 </element>
-<element name="CN1" library="TAStm32_v4" package="CA0612KRX7R7BB104" value="330pF" x="64.5428" y="2.25" smashed="yes" rot="R180">
+<element name="CN1" library="TAStm32_v4" package="CA0612KRX7R7BB104" value="DNP" x="64.5428" y="2.25" smashed="yes" rot="R180">
 <attribute name="DESCRIPTION" value="Phycomp Capacitor Array 100nF 16V dc +/-10% 4-way X7R Dielectric 0612 (1632M) Package C-Array Series Surface Mount" x="64.5428" y="2.25" size="1.778" layer="27" rot="R180" display="off"/>
 <attribute name="HEIGHT" value="0mm" x="64.5428" y="2.25" size="1.778" layer="27" rot="R180" display="off"/>
@@
 <attribute name="VALUE" x="64.5428" y="2.25" size="1.27" layer="27" rot="R180" align="center"/>
 </element>
-<element name="CN2" library="TAStm32_v4" package="CA0612KRX7R7BB104" value="330pF" x="64.5428" y="12" smashed="yes" rot="R180">
+<element name="CN2" library="TAStm32_v4" package="CA0612KRX7R7BB104" value="DNP" x="64.5428" y="12" smashed="yes" rot="R180">
 <attribute name="DESCRIPTION" value="Phycomp Capacitor Array 100nF 16V dc +/-10% 4-way X7R Dielectric 0612 (1632M) Package C-Array Series Surface Mount" x="70.6388" y="12" size="1.778" layer="27" rot="R180" display="off"/>
 <attribute name="HEIGHT" value="0mm" x="70.6388" y="12" size="1.778" layer="27" rot="R180" display="off"/>
@@
 <attribute name="VALUE" x="66.7976" y="19.3168" size="1.016" layer="27" rot="R90"/>
 </element>
-<element name="S2" library="TAStm32_v4" package="3-1825910-1_318259101" package3d_urn="urn:adsk.eagle:package:29257505/2" value="3-1825910-1_SWITCHN" x="66" y="37" smashed="yes">
+<element name="S2" library="TAStm32_v4" package="3-1825910-1_318259101" package3d_urn="urn:adsk.eagle:package:29257505/2" value="3-1825910-1" x="66" y="37" smashed="yes">
 <attribute name="NAME" x="62.0114" y="41.3768" size="1.27" layer="25" align="center"/>
 <attribute name="VALUE" x="66.265" y="37" size="1.27" layer="27" align="center"/>
 </element>
-<element name="S1" library="TAStm32_v4" package="3-1825910-1_318259101" package3d_urn="urn:adsk.eagle:package:29257505/2" value="3-1825910-1_SWITCHN" x="66" y="30" smashed="yes">
+<element name="S1" library="TAStm32_v4" package="3-1825910-1_318259101" package3d_urn="urn:adsk.eagle:package:29257505/2" value="3-1825910-1" x="66" y="30" smashed="yes">
 <attribute name="NAME" x="65.6622" y="25.9948" size="1.27" layer="25" align="center"/>
 <attribute name="VALUE" x="66.265" y="30" size="1.27" layer="27" align="center"/>
 </element>
-<element name="S4" library="TAStm32_v4" package="3-1825910-1_318259101" package3d_urn="urn:adsk.eagle:package:29257505/2" value="3-1825910-1_SWITCHN" x="34" y="37" smashed="yes">
+<element name="S4" library="TAStm32_v4" package="3-1825910-1_318259101" package3d_urn="urn:adsk.eagle:package:29257505/2" value="3-1825910-1" x="34" y="37" smashed="yes">
 <attribute name="NAME" x="34.4174" y="41.572" size="1.27" layer="25" align="center"/>
 <attribute name="VALUE" x="34.265" y="37" size="1.27" layer="27" align="center"/>
 </element>
-<element name="S3" library="TAStm32_v4" package="3-1825910-1_318259101" package3d_urn="urn:adsk.eagle:package:29257505/2" value="3-1825910-1_SWITCHN" x="34" y="30" smashed="yes">
+<element name="S3" library="TAStm32_v4" package="3-1825910-1_318259101" package3d_urn="urn:adsk.eagle:package:29257505/2" value="3-1825910-1" x="34" y="30" smashed="yes">
 <attribute name="NAME" x="33.741" y="25.3852" size="1.27" layer="25" align="center"/>
 <attribute name="VALUE" x="34.265" y="30" size="1.27" layer="27" align="center"/>
@@
 <wire x1="41.4528" y1="35.09094375" x2="41.4528" y2="32.20734375" width="0.1524" layer="1"/>
 <wire x1="38.68345625" y1="29.438" x2="36.4356" y2="29.438" width="0.1524" layer="1"/>
-<wire x1="37.7952" y1="20.4908" x2="37.8516" y2="20.4344" width="0.1524" layer="16"/>
 <via x="37.8516" y="20.4344" extent="1-16" drill="0.35"/>
 <via x="36.862" y="17.5388" extent="1-16" drill="0.35"/>
@@
 <contactref element="R1" pad="1"/>
 <contactref element="J5" pad="3"/>
-<wire x1="45.8596" y1="27.5304" x2="45.8184" y2="27.5304" width="0.1524" layer="1"/>
 <wire x1="45.8436" y1="24.66" x2="48.73" y2="24.66" width="0.1524" layer="1"/>
 <wire x1="45.1104" y1="21.336" x2="44.5008" y2="20.7264" width="0.1524" layer="1"/>
